Commit message: added changes after sessipn with @pat92fr

File: hdumcke_merge_ws/src/my_robot_description/urdf/mech/base.urdf.xacro (robot description, xacro)
@@ -41,5 +41,5 @@
       <parent link="base_footprint"/>
       <child link="base_link"/>
-      <origin xyz="0 0 ${wheel_radius - wheel_pos_z}" rpy="0 0 0"/>
+      <origin xyz="-0.15 0 ${wheel_radius - wheel_pos_z}" rpy="0 0 0"/>
     </joint>
   </xacro:macro>
